File: pcb/Gear80-A_1.0mm/Gear80-A_1.0mm.kicad_pcb (KiCad board)
At the start: 2 copper layers, 388.9 x 93.7 mm, 342 parts, among them J1 Conn_01x04, J2 Conn_01x10_Pin, J3 Conn_01x10_Pin, J4 Conn_01x10_Pin, J5 Conn_01x10_Pin, J6 Conn_01x10_Pin, J7 Conn_01x10_Pin, U1 XC6206P332MR, U3 W25Q128JVSIQ, U4 RP2040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

Commit message: Add files via upload
Parts:
- removed the ? at (348.7, 49.8)
- removed the ? at (52.4, 57.2)
- removed the ? at (52.4, 56.2)
- removed the ? at (52.3, 53.2)
- removed the ? at (348.7, 53.2)
- removed the ? at (58.2, 55.2)
- removed the ? at (58.2, 50.2)
- removed the ? at (52.3, 50.2)
- removed the ? at (52.3, 49.2)
- removed the ? at (342.8, 53.2)
- removed the ? at (52.3, 51.8)
- removed the ? at (52.3, 57.8)
- removed the ? at (342.8, 50.2)
- removed the ? at (342.8, 50.8)
- removed the ? at (52.3, 53.8)
- removed the ? at (52.3, 55.2)
- removed the ? at (348.7, 53.8)
- removed the ? at (342.8, 54.2)
- removed the ? at (58.2, 54.2)
- removed the ? at (52.3, 50.8)
- removed the ? at (58.2, 53.2)
- removed the ? at (58.2, 49.8)
- removed the ? at (348.7, 57.8)
- removed the ? at (348.7, 54.8)
- removed the ? at (52.3, 54.2)
- removed the ? at (52.3, 52.8)
- removed the ? at (52.3, 49.8)
- removed the ? at (348.7, 56.8)
- removed the ? at (58.2, 53.8)
- removed the ? at (58.2, 50.8)
- removed the ? at (342.8, 49.8)
- removed the ? at (58.2, 52.8)
- removed the ? at (58.2, 51.8)
- removed the ? at (58.2, 48.8)
- removed the ? at (342.8, 52.8)
- removed the ? at (342.8, 51.2)
- removed the ? at (348.7, 51.2)
- removed the ? at (348.7, 48.2)
- removed the ? at (342.8, 52.1)
- removed the ? at (348.7, 51.8)
- removed the ? at (342.9, 57.2)
- removed the ? at (52.4, 55.8)
- removed the ? at (58.2, 51.2)
- removed the ? at (58.2, 57.2)
- removed the ? at (342.9, 56.2)
- removed the ? at (342.8, 53.8)
- removed the ? at (342.8, 49.2)
- removed the ? at (348.7, 52.8)
- removed the ? at (58.2, 56.2)
- removed the ? at (58.2, 49.2)
- removed the ? at (348.7, 55.8)
- removed the ? at (58.2, 56.8)
- removed the ? at (348.7, 54.2)
- removed the ? at (348.7, 52.1)
- removed the ? at (348.7, 55.2)
- removed the ? at (58.2, 57.8)
- removed the ? at (342.9, 56.8)
- removed the ? at (58.2, 54.8)
- removed the ? at (342.9, 54.8)
- removed the ? at (58.2, 48.2)
- removed the ? at (348.7, 48.8)
- removed the ? at (348.7, 56.2)
- removed the ? at (52.3, 54.8)
- removed the ? at (52.3, 51.2)
- removed the ? at (348.7, 50.8)
- removed the ? at (342.8, 48.2)
- removed the ? at (348.7, 50.2)
- removed the ? at (52.3, 48.8)
- removed the ? at (58.2, 52.2)
- removed the ? at (52.4, 56.8)
- removed the ? at (348.7, 57.2)
- removed the ? at (342.9, 55.2)
- removed the ? at (342.8, 57.8)
- removed the ? at (342.9, 55.8)
- removed the ? at (52.3, 52.2)
- removed the ? at (348.7, 49.2)
- removed the ? at (58.2, 55.8)
- removed the ? at (342.8, 51.8)
- removed the ? at (342.8, 48.8)
- added ?: , , F.Cu at (58.1, 57.1)
- added ?: , , F.Cu at (342.9, 54.1)
- added ?: , , F.Cu at (58.1, 49.0)
- added ?: , , F.Cu at (342.9, 48.0)
- added ?: , , F.Cu at (52.4, 50.1)
- added ?: , , F.Cu at (348.4, 52.0)
- added ?: , , F.Cu at (348.4, 53.0)
- added ?: , , F.Cu at (52.4, 52.0)
- added ?: , , F.Cu at (58.1, 52.0)
- added ?: , , F.Cu at (348.4, 51.1)
- added ?: , , F.Cu at (58.1, 57.9)
- added ?: , , F.Cu at (342.9, 50.1)
- added ?: , , F.Cu at (58.1, 53.0)
- added ?: , , F.Cu at (342.9, 55.1)
- added ?: , , F.Cu at (52.4, 56.1)
- added ?: , , F.Cu at (342.9, 56.1)
- added ?: , , F.Cu at (52.4, 49.0)
- added ?: , , F.Cu at (348.4, 48.0)
- added ?: , , F.Cu at (342.9, 57.9)
- added ?: , , F.Cu at (348.4, 57.9)
- added ?: , , F.Cu at (348.4, 55.1)
- added ?: , , F.Cu at (58.1, 54.1)
- added ?: , , F.Cu at (52.4, 57.9)
- added ?: , , F.Cu at (348.4, 57.1)
- added ?: , , F.Cu at (52.4, 55.1)
- added ?: , , F.Cu at (348.4, 50.1)
- added ?: , , F.Cu at (348.4, 56.1)
- added ?: , , F.Cu at (58.1, 50.1)
- added ?: , , F.Cu at (58.1, 51.1)
- added ?: , , F.Cu at (348.4, 54.1)
- added ?: , , F.Cu at (58.1, 55.1)
- added ?: , , F.Cu at (342.9, 51.1)
- added ?: , , F.Cu at (342.9, 49.0)
- added ?: , , F.Cu at (58.1, 56.1)
- added ?: , , F.Cu at (342.9, 52.0)
- added ?: , , F.Cu at (52.4, 54.1)
- added ?: , , F.Cu at (342.9, 57.1)
- added ?: , , F.Cu at (342.9, 53.0)
- added ?: , , F.Cu at (52.4, 53.0)
- added ?: , , F.Cu at (348.4, 49.0)
- added ?: , , F.Cu at (52.4, 57.1)
- added ?: , , F.Cu at (58.1, 48.0)
- added ?: , , F.Cu at (52.4, 51.1)
- moved ? 0.18 mm to (52.4, 48.0)

Commit message: Add files via upload
Connections:
- MX63 pad 1: Net-(D48-A) -> COL0
- MX73 pad 2: Net-(D48-A) -> COL0
- MX82 pad 1: Net-(D48-A) -> COL0
Routing:
- net COL0: track 198.4 -> 233.2 mm
- net Net-(D48-A): track 61.4 -> 30.7 mm

Commit message: Add files via upload
Parts:
- added MX113: MX_SW_solder, PCM_marbastlib-mx:SW_MX_1u, F.Cu at (155.3, 100.0)
- added MX114: MX_SW_solder, PCM_marbastlib-mx:SW_MX_1u, F.Cu at (245.7, 100.0)
- added MX115: MX_SW_solder, PCM_marbastlib-mx:SW_MX_1u, F.Cu at (212.4, 100.0)
- moved D67 5.61 mm to (219.7, 101.4), turned to 90 degrees
- moved D68 5.58 mm to (248.2, 104.5)
- moved D66 4.42 mm to (167.5, 101.4)
- moved C9 1.16 mm to (172.6, 96.4), turned to 180 degrees
- moved G*** 0.40 mm to (228.3, 96.2)
- turned MX66 to 180 degrees
- turned MX67 to 0 degrees
Connections:
- MX66 pad 1: COL5 -> Net-(D66-A)
- MX66 pad 2: Net-(D66-A) -> COL5
- MX67 pad 1: Net-(D67-A) -> COL7
- MX67 pad 2: COL7 -> Net-(D67-A)
Routing:
- net COL9: track 156.2 -> 168.5 mm
- net Net-(D66-A): track 4.36 -> 15.3 mm
- net Net-(D68-A): track 4.36 -> 13.7 mm
- net COL5: track 119.4 -> 127.8 mm, vias 0 -> 1
- net Net-(D67-A): track 29.3 -> 35.2 mm
- net COL10: track 180.4 -> 174.9 mm
- net COL4: track 119.9 -> 124.9 mm
- net COL1: track 192.8 -> 188.6 mm
- net COL7: track 134.2 -> 137.6 mm
- net COL3: track 140.3 -> 137.4 mm
- net COL2: track 179.1 -> 176.3 mm
- net +3V3: track 146.4 -> 144.1 mm
- net COL14: track 319.1 -> 321.4 mm
- net COL11: track 207.5 -> 209.8 mm
- net COL12: track 261.1 -> 263.4 mm
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