File: pcb/Gear80-A_1.0mm/Gear80-A_1.0mm.kicad_pcb (KiCad board)
At the start: 2 copper layers, 388.9 x 93.7 mm, 309 parts, among them J1 Conn_01x04, J2 Conn_01x10_Pin, J3 Conn_01x10_Pin, J4 Conn_01x10_Pin, J5 Conn_01x10_Pin, J6 Conn_01x10_Pin, J7 Conn_01x10_Pin, U1 XC6206P332MR, U3 W25Q128JVSIQ, U4 RP2040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

Commit message: Add files via upload
Routing:
- net COL19: track 534.2 -> 536.4 mm

Commit message: Add files via upload
Routing:
- net COL19: track 536.4 -> 522.1 mm, vias 7 -> 9

Commit message: Add files via upload
Parts:
- C5: value 10u -> 100n; footprint Capacitor_SMD:C_0603_1608Metric -> Capacitor_SMD:C_0402_1005Metric
- moved C5 0.54 mm to (175.0, 84.7)
Routing:
- net +3V3: track 144.1 -> 143.2 mm
- net GND: track 86.2 -> 85.6 mm
