File: pcb/Gear80-A_1.0mm/Gear80-A_1.0mm.kicad_sch (KiCad schematic)
At the start: 249 parts, among them J2 Conn_01x10_Pin, J3 Conn_01x04, J3 Conn_01x10_Pin, J4 Conn_01x10_Pin, J5 Conn_01x10_Pin, J6 Conn_01x10_Pin, J7 Conn_01x10_Pin, U1 XC6206P332MR, U3 W25Q128JVSIQ, U4 RP2040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

Commit message: Add files via upload
Connections:
- net COL0: now also MX63.1, MX73.2, MX82.1
- net at D48.2 (A), MX47.2, MX48.2: no longer MX63.1, MX73.2, MX82.1
Changed lines of the file:
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@@
   (junction (at 398.78 182.88) (diameter 0) (color 0 0 0 0)
   )
-  (junction (at 356.87 162.56) (diameter 0) (color 0 0 0 0)
-  )
   (junction (at 568.96 120.65) (diameter 0) (color 0 0 0 0)
   )
+  (junction (at 52.07 177.8) (diameter 0) (color 0 0 0 0)
+  )
+  (junction (at 534.67 92.71) (diameter 0) (color 0 0 0 0)
+  )
+  (junction (at 356.87 137.16) (diameter 0) (color 0 0 0 0)
+  )
+  (junction (at 415.29 135.89) (diameter 0) (color 0 0 0 0)
+  )
+  (junction (at 459.74 157.48) (diameter 0) (color 0 0 0 0)
+  )
+  (junction (at 660.4 111.76) (diameter 0) (color 0 0 0 0)
+  )
+  (junction (at 509.27 168.91) (diameter 0) (color 0 0 0 0)
+  )
+  (junction (at 254 93.98) (diameter 0) (color 0 0 0 0)
+  )
+  (junction (at 393.7 177.8) (diameter 0) (color 0 0 0 0)
+  )
+  (junction (at 391.16 147.32) (diameter 0) (color 0 0 0 0)
+  )
+  (junction (at 464.82 168.91) (diameter 0) (color 0 0 0 0)
+  )
+  (junction (at 563.88 115.57) (diameter 0) (color 0 0 0 0)
+  )
+  (junction (at 254 115.57) (diameter 0) (color 0 0 0 0)
+  )
+  (junction (at 420.37 147.32) (diameter 0) (color 0 0 0 0)
+  )
+  (junction (at 66.04 22.86) (diameter 0) (color 0 0 0 0)
+  )
+  (junction (at 554.99 127) (diameter 0) (color 0 0 0 0)
+  )
+  (junction (at 391.16 168.91) (diameter 0) (color 0 0 0 0)
+  )
+  (junction (at 504.19 157.48) (diameter 0) (color 0 0 0 0)
+  )
+  (junction (at 391.16 104.14) (diameter 0) (color 0 0 0 0)
+  )
+  (junction (at 490.22 157.48) (diameter 0) (color 0 0 0 0)
+  )
+  (junction (at 118.11 142.24) (diameter 0) (color 0 0 0 0)
+  )
+  (junction (at 372.11 115.57) (diameter 0) (color 0 0 0 0)
+  )
+  (junction (at 361.95 189.23) (diameter 0) (color 0 0 0 0)
+  )
+  (junction (at 391.16 127) (diameter 0) (color 0 0 0 0)
+  )
+  (junction (at 77.47 254) (diameter 0) (color 0 0 0 0)
+  )
+  (junction (at 406.4 147.32) (diameter 0) (color 0 0 0 0)
+  )
+  (junction (at 377.19 168.91) (diameter 0) (color 0 0 0 0)
+  )
+  (junction (at 88.9 142.24) (diameter 0) (color 0 0 0 0)
+  )
+  (junction (at 490.22 92.71) (diameter 0) (color 0 0 0 0)
+  )
+  (junction (at 78.74 149.86) (diameter 0) (color 0 0 0 0)
+  )
+  (junction (at 539.75 189.23) (diameter 0) (color 0 0 0 0)
+  )
+  (junction (at 678.18 154.94) (diameter 0) (color 0 0 0 0)
+  )
+  (junction (at 36.83 142.24) (diameter 0) (color 0 0 0 0)
+  )
+  (junction (at 361.95 182.88) (diameter 0) (color 0 0 0 0)
+  )
+  (junction (at 549.91 92.71) (diameter 0) (color 0 0 0 0)
+  )
+  (junction (at 495.3 104.14) (diameter 0) (color 0 0 0 0)
+  )
+  (junction (at 509.27 189.23) (diameter 0) (color 0 0 0 0)
+  )
+  (junction (at 459.74 92.71) (diameter 0) (color 0 0 0 0)
+  )
+  (junction (at 563.88 157.48) (diameter 0) (color 0 0 0 0)
+  )
+  (junction (at 459.74 115.57) (diameter 0) (color 0 0 0 0)
+  )
+  (junction (at 361.95 127) (diameter 0) (color 0 0 0 0)
+  )
+  (junction (at 123.19 149.86) (diameter 0) (color 0 0 0 0)
+  )
+  (junction (at 539.75 182.88) (diameter 0) (color 0 0 0 0)
+  )
   (junction (at 361.95 162.56) (diameter 0) (color 0 0 0 0)
-  )
-  (junction (at 52.07 177.8) (diameter 0) (color 0 0 0 0)
-  )
-  (junction (at 534.67 92.71) (diameter 0) (color 0 0 0 0)
-  )
-  (junction (at 356.87 137.16) (diameter 0) (color 0 0 0 0)
-  )
-  (junction (at 415.29 135.89) (diameter 0) (color 0 0 0 0)
-  )
-  (junction (at 459.74 157.48) (diameter 0) (color 0 0 0 0)
-  )
-  (junction (at 660.4 111.76) (diameter 0) (color 0 0 0 0)
-  )
-  (junction (at 509.27 168.91) (diameter 0) (color 0 0 0 0)
-  )
-  (junction (at 254 93.98) (diameter 0) (color 0 0 0 0)
-  )
-  (junction (at 393.7 177.8) (diameter 0) (color 0 0 0 0)
-  )
-  (junction (at 391.16 147.32) (diameter 0) (color 0 0 0 0)
-  )
-  (junction (at 464.82 168.91) (diameter 0) (color 0 0 0 0)
-  )
-  (junction (at 563.88 115.57) (diameter 0) (color 0 0 0 0)
-  )
-  (junction (at 254 115.57) (diameter 0) (color 0 0 0 0)
-  )
-  (junction (at 420.37 147.32) (diameter 0) (color 0 0 0 0)
-  )
-  (junction (at 66.04 22.86) (diameter 0) (color 0 0 0 0)
-  )
-  (junction (at 554.99 127) (diameter 0) (color 0 0 0 0)
-  )
-  (junction (at 391.16 168.91) (diameter 0) (color 0 0 0 0)
-  )
-  (junction (at 504.19 157.48) (diameter 0) (color 0 0 0 0)
-  )
-  (junction (at 391.16 104.14) (diameter 0) (color 0 0 0 0)
-  )
-  (junction (at 490.22 157.48) (diameter 0) (color 0 0 0 0)
-  )
-  (junction (at 118.11 142.24) (diameter 0) (color 0 0 0 0)
-  )
-  (junction (at 372.11 115.57) (diameter 0) (color 0 0 0 0)
-  )
-  (junction (at 361.95 189.23) (diameter 0) (color 0 0 0 0)
-  )
-  (junction (at 391.16 127) (diameter 0) (color 0 0 0 0)
-  )
-  (junction (at 77.47 254) (diameter 0) (color 0 0 0 0)
-  )
-  (junction (at 406.4 147.32) (diameter 0) (color 0 0 0 0)
-  )
-  (junction (at 377.19 168.91) (diameter 0) (color 0 0 0 0)
-  )
-  (junction (at 88.9 142.24) (diameter 0) (color 0 0 0 0)
-  )
-  (junction (at 490.22 92.71) (diameter 0) (color 0 0 0 0)
-  )
-  (junction (at 78.74 149.86) (diameter 0) (color 0 0 0 0)
-  )
-  (junction (at 539.75 189.23) (diameter 0) (color 0 0 0 0)
-  )
-  (junction (at 678.18 154.94) (diameter 0) (color 0 0 0 0)
-  )
-  (junction (at 36.83 142.24) (diameter 0) (color 0 0 0 0)
-  )
-  (junction (at 361.95 182.88) (diameter 0) (color 0 0 0 0)
-  )
-  (junction (at 549.91 92.71) (diameter 0) (color 0 0 0 0)
-  )
-  (junction (at 495.3 104.14) (diameter 0) (color 0 0 0 0)
-  )
-  (junction (at 509.27 189.23) (diameter 0) (color 0 0 0 0)
-  )
-  (junction (at 459.74 92.71) (diameter 0) (color 0 0 0 0)
-  )
-  (junction (at 563.88 157.48) (diameter 0) (color 0 0 0 0)
-  )
-  (junction (at 459.74 115.57) (diameter 0) (color 0 0 0 0)
-  )
-  (junction (at 361.95 127) (diameter 0) (color 0 0 0 0)
-  )
-  (junction (at 123.19 149.86) (diameter 0) (color 0 0 0 0)
-  )
-  (junction (at 539.75 182.88) (diameter 0) (color 0 0 0 0)
   )
   (junction (at 449.58 127) (diameter 0) (color 0 0 0 0)
@@
     (stroke (width 0) (type default))
   )
-  (wire (pts (xy 356.87 162.56) (xy 361.95 162.56))
-    (stroke (width 0) (type default))
-  )
   (wire (pts (xy 361.95 127) (xy 377.19 127))
     (stroke (width 0) (type default))
@@
     (stroke (width 0) (type default))
   )
-  (wire (pts (xy 356.87 162.56) (xy 356.87 177.8))
+  (wire (pts (xy 356.87 157.48) (xy 356.87 177.8))
     (stroke (width 0) (type default))
   )
@@
     (stroke (width 0) (type default))
   )
-  (wire (pts (xy 354.33 162.56) (xy 356.87 162.56))
-    (stroke (width 0) (type default))
-  )
   (wire (pts (xy 524.51 147.32) (xy 539.75 147.32))
     (stroke (width 0) (type default))
@@
     (stroke (width 0) (type default))
   )
+  (wire (pts (xy 354.33 162.56) (xy 361.95 162.56))
+    (stroke (width 0) (type default))
+  )

Commit message: Add files via upload
Parts:
- added MX113, MX114, MX115: MX_SW_solder, PCM_marbastlib-mx:SW_MX_1u, symbol PCM_marbastlib-mx:MX_SW_HS
Connections:
- net COL5: now also MX66.2, MX113.1; no longer MX66.1
- net COL7: now also MX67.1, MX115.2; no longer MX67.2
- net COL9: now also MX114.1
- net at D66.2 (A): now also MX66.1, MX113.2; no longer MX66.2
- net at D67.2 (A), MX76.2, MX83.2: now also MX67.2, MX115.1; no longer MX67.1
- net at D68.2 (A), MX68.2: now also MX114.2
Other:
- moved on the sheet: MX66, MX67, MX68, MX76

Commit message: Add files via upload
Parts:
- C5: value 10u -> 100n; footprint Capacitor_SMD:C_0603_1608Metric -> Capacitor_SMD:C_0402_1005Metric
Changed lines of the file:
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@@
-    )
-  )
-  (symbol (lib_id "Device:C_Small") (at 118.11 146.05 0) (unit 1)
-    (in_bom yes) (on_board yes) (dnp no) (fields_autoplaced)
-    (property "Reference" "C5" (at 120.65 144.7863 0)
-      (effects (font (size 1.27 1.27)) (justify left))
-    )
-    (property "Value" "10u" (at 120.65 147.3263 0)
-      (effects (font (size 1.27 1.27)) (justify left))
-    )
-    (property "Footprint" "Capacitor_SMD:C_0603_1608Metric" (at 118.11 146.05 0)
-      (effects (font (size 1.27 1.27)) hide)
-    )
-    (property "Datasheet" "~" (at 118.11 146.05 0)
-      (effects (font (size 1.27 1.27)) hide)
-    )
-    (pin "1")
-    (pin "2")
-    (instances
-      (project "Gear80-A_1.0mm"
-        (path "/b7ecd40f-fbd1-4363-aa36-fbfbff6aee59"
-          (reference "C5") (unit 1)
-        )
-      )
     )
   )
@@
         )
       )
+    )
+  )
+  (symbol (lib_id "Device:C_Small") (at 118.11 146.05 0) (unit 1)
+    (in_bom yes) (on_board yes) (dnp no) (fields_autoplaced)
+    (property "Reference" "C5" (at 120.65 144.7863 0)
+      (effects (font (size 1.27 1.27)) (justify left))
+    )
+    (property "Value" "100n" (at 120.65 147.3263 0)
+      (effects (font (size 1.27 1.27)) (justify left))
+    )
+    (property "Footprint" "Capacitor_SMD:C_0402_1005Metric" (at 118.11 146.05 0)
+      (effects (font (size 1.27 1.27)) hide)
+    )
+    (property "Datasheet" "~" (at 118.11 146.05 0)
+      (effects (font (size 1.27 1.27)) hide)
+    )
+    (pin "1")
+    (pin "2")
+    (instances
+      (project "Gear80-A_1.0mm"
+        (path "/b7ecd40f-fbd1-4363-aa36-fbfbff6aee59"
+          (reference "C5") (unit 1)
+        )
+      )
