File: pcb/Gear80-A_0.5mm/Gear80-A_0.5mm.kicad_pcb (KiCad board)
At the start: 2 copper layers, 388.9 x 93.7 mm, 250 parts, among them J1 Conn_01x04, J2 Conn_01x10_Pin, J3 Conn_01x10_Pin, J4 Conn_01x10_Pin, J5 Conn_01x10_Pin, J6 Conn_01x10_Pin, J7 Conn_01x10_Pin, U1 XC6206P332MR, U3 W25Q128JVSIQ, U4 RP2040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

Commit message: Add files via upload
Connections:
- MX63 pad 1: Net-(D48-A) -> COL0
- MX73 pad 2: Net-(D48-A) -> COL0
- MX82 pad 1: Net-(D48-A) -> COL0
Routing:
- net COL0: track 198.4 -> 233.2 mm
- net Net-(D48-A): track 61.4 -> 30.7 mm

Commit message: Add files via upload
Parts:
- added MX113: MX_SW_solder, PCM_marbastlib-mx:SW_MX_1u, F.Cu at (155.3, 100.0)
- added MX114: MX_SW_solder, PCM_marbastlib-mx:SW_MX_1u, F.Cu at (212.4, 100.0)
- added MX115: MX_SW_solder, PCM_marbastlib-mx:SW_MX_1u, F.Cu at (245.7, 100.0)
- moved D67 5.88 mm to (219.9, 101.2), turned to 90 degrees
- moved D68 5.42 mm to (248.1, 104.3)
- moved D66 4.42 mm to (167.5, 101.4)
- moved C9 1.47 mm to (172.2, 96.4), turned to 180 degrees
- turned MX66 to 180 degrees
- turned MX67 to 0 degrees
Connections:
- MX66 pad 1: COL5 -> Net-(D66-A)
- MX66 pad 2: Net-(D66-A) -> COL5
- MX67 pad 1: Net-(D67-A) -> COL7
- MX67 pad 2: COL7 -> Net-(D67-A)
Routing:
- net COL9: track 156.2 -> 168.2 mm
- net Net-(D66-A): track 4.36 -> 15.3 mm
- net Net-(D68-A): track 4.36 -> 13.6 mm
- net COL5: track 119.4 -> 127.5 mm, vias 0 -> 1
- net COL1: track 192.8 -> 187.6 mm
- net COL0: track 233.2 -> 228.2 mm
- net Net-(D67-A): track 29.3 -> 34.3 mm
- net COL10: track 180.4 -> 175.7 mm
- net COL7: track 134.2 -> 138.7 mm
- net COL2: track 179.1 -> 175.4 mm
- net COL3: track 140.3 -> 136.6 mm
- net COL19: track 336.7 -> 333.3 mm
- net COL14: track 319.1 -> 321.4 mm
- net COL11: track 207.5 -> 209.8 mm
- net COL12: track 261.1 -> 263.4 mm
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
Commit message: Add files via upload
Parts:
- C5: value 10u -> 100n; footprint Capacitor_SMD:C_0603_1608Metric -> Capacitor_SMD:C_0402_1005Metric
- moved C5 0.05 mm to (175.3, 84.2)
Routing:
- net GND: track 86.3 -> 85.7 mm
- net +3V3: track 144.3 -> 143.7 mm
