File: pcb/Gear80-A_0.5mm/Gear80-A_0.5mm.kicad_pcb (KiCad board)
At the start: 2 copper layers, 388.9 x 93.7 mm, 253 parts, among them J1 Conn_01x04, J2 Conn_01x10_Pin, J3 Conn_01x10_Pin, J4 Conn_01x10_Pin, J5 Conn_01x10_Pin, J6 Conn_01x10_Pin, J7 Conn_01x10_Pin, U1 XC6206P332MR, U3 W25Q128JVSIQ, U4 RP2040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

Commit message: Add files via upload
Routing:
- net COL7: track 138.7 -> 137.8 mm
- net GND: vias 24 -> 25
