File: pcb/Gear80-A_0.5mm/Gear80-A_0.5mm.kicad_sch (KiCad schematic)
At the start: 249 parts, among them J2 Conn_01x10_Pin, J3 Conn_01x04, J3 Conn_01x10_Pin, J4 Conn_01x10_Pin, J5 Conn_01x10_Pin, J6 Conn_01x10_Pin, J7 Conn_01x10_Pin, U1 XC6206P332MR, U3 W25Q128JVSIQ, U4 RP2040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

Commit message: Add files via upload
Connections:
- net COL0: now also MX63.1, MX73.2, MX82.1
- net at D48.2 (A), MX47.2, MX48.2: no longer MX63.1, MX73.2, MX82.1
Changed lines of the file:
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@@
   (junction (at 665.48 181.61) (diameter 0) (color 0 0 0 0)
   )
+  (junction (at 361.95 162.56) (diameter 0) (color 0 0 0 0)
+  )
   (junction (at 534.67 135.89) (diameter 0) (color 0 0 0 0)
   )
@@
   (junction (at 398.78 182.88) (diameter 0) (color 0 0 0 0)
   )
-  (junction (at 356.87 162.56) (diameter 0) (color 0 0 0 0)
-  )
   (junction (at 568.96 120.65) (diameter 0) (color 0 0 0 0)
-  )
-  (junction (at 361.95 162.56) (diameter 0) (color 0 0 0 0)
   )
   (junction (at 259.08 187.96) (diameter 0) (color 0 0 0 0)
@@
     (stroke (width 0) (type default))
   )
-  (wire (pts (xy 356.87 162.56) (xy 361.95 162.56))
-    (stroke (width 0) (type default))
-  )
   (wire (pts (xy 361.95 127) (xy 377.19 127))
     (stroke (width 0) (type default))
@@
     (stroke (width 0) (type default))
   )
-  (wire (pts (xy 356.87 162.56) (xy 356.87 177.8))
-    (stroke (width 0) (type default))
-  )
   (wire (pts (xy 665.48 143.51) (xy 683.26 143.51))
     (stroke (width 0) (type default))
@@
     (stroke (width 0) (type default))
   )
+  (wire (pts (xy 354.33 162.56) (xy 361.95 162.56))
+    (stroke (width 0) (type default))
+  )
   (wire (pts (xy 509.27 104.14) (xy 524.51 104.14))
     (stroke (width 0) (type default))
@@
     (stroke (width 0) (type default))
   )
-  (wire (pts (xy 354.33 162.56) (xy 356.87 162.56))
-    (stroke (width 0) (type default))
-  )
   (wire (pts (xy 524.51 147.32) (xy 539.75 147.32))
     (stroke (width 0) (type default))
@@
     (stroke (width 0) (type default))
   )
+  (wire (pts (xy 356.87 157.48) (xy 356.87 177.8))
+    (stroke (width 0) (type default))
+  )

Commit message: Add files via upload
Parts:
- added MX113, MX114, MX115: MX_SW_solder, PCM_marbastlib-mx:SW_MX_1u, symbol PCM_marbastlib-mx:MX_SW_HS
Connections:
- net COL5: now also MX66.2, MX113.1; no longer MX66.1
- net COL7: now also MX67.1, MX114.2; no longer MX67.2
- net COL9: now also MX115.1
- net at D66.2 (A): now also MX66.1, MX113.2; no longer MX66.2
- net at D67.2 (A), MX76.2, MX83.2: now also MX67.2, MX114.1; no longer MX67.1
- net at D68.2 (A), MX68.2: now also MX115.2
Other:
- moved on the sheet: MX66, MX67

Commit message: Add files via upload
Parts:
- C5: value 10u -> 100n; footprint Capacitor_SMD:C_0603_1608Metric -> Capacitor_SMD:C_0402_1005Metric
Changed lines of the file:
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@@
+    )
+  )
+  (symbol (lib_id "Device:C_Small") (at 118.11 146.05 0) (unit 1)
+    (in_bom yes) (on_board yes) (dnp no) (fields_autoplaced)
+    (property "Reference" "C5" (at 120.65 144.7863 0)
+      (effects (font (size 1.27 1.27)) (justify left))
+    )
+    (property "Value" "100n" (at 120.65 147.3263 0)
+      (effects (font (size 1.27 1.27)) (justify left))
+    )
+    (property "Footprint" "Capacitor_SMD:C_0402_1005Metric" (at 118.11 146.05 0)
+      (effects (font (size 1.27 1.27)) hide)
+    )
+    (property "Datasheet" "~" (at 118.11 146.05 0)
+      (effects (font (size 1.27 1.27)) hide)
+    )
+    (pin "1")
+    (pin "2")
+    (instances
+      (project "Gear80-A_0.5mm"
+        (path "/b7ecd40f-fbd1-4363-aa36-fbfbff6aee59"
+          (reference "C5") (unit 1)
+        )
+      )
     )
   )
@@
         )
       )
-    )
-  )
-  (symbol (lib_id "Device:C_Small") (at 118.11 146.05 0) (unit 1)
-    (in_bom yes) (on_board yes) (dnp no) (fields_autoplaced)
-    (property "Reference" "C5" (at 120.65 144.7863 0)
-      (effects (font (size 1.27 1.27)) (justify left))
-    )
-    (property "Value" "10u" (at 120.65 147.3263 0)
-      (effects (font (size 1.27 1.27)) (justify left))
-    )
-    (property "Footprint" "Capacitor_SMD:C_0603_1608Metric" (at 118.11 146.05 0)
-      (effects (font (size 1.27 1.27)) hide)
-    )
-    (property "Datasheet" "~" (at 118.11 146.05 0)
-      (effects (font (size 1.27 1.27)) hide)
-    )
-    (pin "1")
-    (pin "2")
-    (instances
-      (project "Gear80-A_0.5mm"
-        (path "/b7ecd40f-fbd1-4363-aa36-fbfbff6aee59"
-          (reference "C5") (unit 1)
-        )
-      )
