File: pcb/Gear80 solder/Gear80 solder.kicad_pcb (KiCad board)
At the start: 2 copper layers, 388.9 x 93.7 mm, 207 parts, among them J3 Conn_01x04, U1 RP2040, U3 W25Q128JVSIQ, U4 XC6206P332MR, Y1 X322512MSB4SI

Commit message: Add files via upload
Routing:
- net COL2: track 390.6 -> 386.4 mm

Commit message: Add files via upload
Parts:
- C4: value 10u -> 100n; footprint Capacitor_SMD:C_0603_1608Metric -> Capacitor_SMD:C_0402_1005Metric
- moved C4 0.29 mm to (192.9, 181.5)
Routing:
- net GND: track 79.0 -> 77.4 mm

Commit message: Add files via upload
Parts:
- moved J3 0.99 mm to (42.2, 152.5)
Routing:
- net +5V: track 163.6 -> 164.8 mm
- net USB_D+: track 178.1 -> 179.0 mm
- net USB_D-: track 176.3 -> 177.0 mm
- net GND: vias 21 -> 22
