File: pcb/gear80_hotswap_flex_cut/gear80_hotswap_flex_cut.kicad_pcb (KiCad board)
At the start: 2 copper layers, 393.7 x 101 mm, 237 parts, among them J1 Conn_01x04, J2 USB_C_Receptacle_USB2.0, J3 SWD, J4 Conn_01x04, J5 USB_C_Receptacle_USB2.0, J8 Conn_01x05, U1 RP2040, U2 XC6206P332MR, U3 W25Q128JVSIQ, U4 SRV05-4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

Commit message: Add files via upload
Parts:
- F1, F2: value MF-MSMF050-2 500mA -> MF-MSMF050-2; footprint Fuse:Fuse_2010_5025Metric -> Fuse:Fuse_1812_4532Metric
