File: pcb/gear80_hotswap_flex_cut/gear80_hotswap_flex_cut.kicad_sch (KiCad schematic)
At the start: 219 parts, among them J1 USB_C_Receptacle_USB2.0, J3 Conn_01x04, J3 SWD, J4 Conn_01x04, J8 Conn_01x05, U1 RP2040, U2 SRV05-4, U2 XC6206P332MR, U3 W25Q128JVSIQ, Y1 X322512MSB4SI

Commit message: Add files via upload
Parts:
- removed F1 (x2): MF-MSMF050-2 500mA, Fuse:Fuse_2010_5025Metric, symbol Leonardo_Rev3e:L-EUL1812
- added F1 (x2): MF-MSMF050-2, Fuse:Fuse_1812_4532Metric, symbol Leonardo_Rev3e:L-EUL1812
Connections:
- net +5V: now also F1.1
- net +5VA: now also F1.1
- net VBUS: now also F1.2
- net VCC: now also F1.2
