File: pcb/gear85_hotswap_flex_cut, number pad/gear85_hotswap_flex_cut, number pad.kicad_sch (KiCad schematic)
At the start: 314 parts, among them J1 USB_C_Receptacle_USB2.0, J11 Conn_01x05, J3 Conn_01x04, J3 SWD, J4 Conn_01x04, J6 Conn_01x10_Pin, J7 Conn_01x10_Pin, J8 Conn_01x05, U1 RP2040, U2 SRV05-4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

Commit message: Add files via upload
Connections:
- net +5V: now also J3.1 (Pin_1); no longer J3.4 (Pin_4)
- net +5VA: now also J4.4 (Pin_4); no longer J4.1 (Pin_1)
- net +5VR: now also J3.1 (Pin_1); no longer J3.4 (Pin_4)
- net GND: now also J3.4 (Pin_4); no longer J3.1 (Pin_1)
- net GNDA: now also J4.1 (Pin_1); no longer J4.4 (Pin_4)
- net GNDR: now also J3.4 (Pin_4); no longer J3.1 (Pin_1)
- net USB_D+: now also J3.3 (Pin_3); no longer J3.2 (Pin_2)
- net USB_D+_DB: now also J4.2 (Pin_2); no longer J4.3 (Pin_3)
- net USB_D+_R: now also J3.3 (Pin_3); no longer J3.2 (Pin_2)
- net USB_D-: now also J3.2 (Pin_2); no longer J3.3 (Pin_3)
- net USB_D-_DB: now also J4.3 (Pin_3); no longer J4.2 (Pin_2)
- net USB_D-_R: now also J3.2 (Pin_2); no longer J3.3 (Pin_3)

Commit message: Add files via upload
Connections:
- net GND2 is gone; now on net GNDR: R3.2, R4.2
Changed lines of the file:
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@@
 	)
 	(symbol
-		(lib_id "power:GND2")
+		(lib_name "GNDA_1")
+		(lib_id "power:GNDA")
 		(at 431.8 218.44 0)
 		(unit 1)
@@
 			)
 		)
-		(property "Value" "GND2"
+		(property "Value" "GNDR"
 			(at 431.8 223.52 0)
 			(effects
